Commit message: Add Map My World project
Added RGBD camera to robot; linked to rtab_ros database file with mapping data; added launch files for mapping/localization

File: my_robot/urdf/board_bot.xacro (robot description, xacro)
@@ -153,5 +153,5 @@
   <!-- Camera -->
   <joint name="camera_joint" type="fixed">
-    <origin xyz="0.5 0 0" rpy="0 0 0"/>
+    <origin xyz="0.5 0 0.025" rpy="0 0 0"/>
     <parent link="body"/>
     <child link="camera"/>
@@ -162,5 +162,5 @@
       <origin xyz="0 0 0" rpy="0 0 0"/>
       <geometry>
-        <sphere radius="0.03" />
+        <sphere radius="0.025" />
       </geometry>
     </visual>
@@ -168,5 +168,5 @@
       <origin xyz="0 0 0" rpy="0 0 0"/>
       <geometry>
-        <sphere radius="0.03" />
+        <sphere radius="0.025" />
       </geometry>
     </collision>
@@ -177,4 +177,30 @@
     </inertial>
   </link>
+ <!-- RGBD Camera -->
+  <joint name="rgbd_camera_optical_joint" type="fixed">
+    <origin xyz="0.5 0 -0.025" rpy="0 0 0"/>
+    <parent link="body"/>
+    <child link="rgbd_camera"/>
+    <axis xyz="0 1 0" rpy="0 0 0"/>
+  </joint>
+  <link name="rgbd_camera">
+    <visual name="rgbd_camera_visual">
+      <origin xyz="0 0 0" rpy="0 0 0"/>
+      <geometry>
+        <sphere radius="0.025" />
+      </geometry>
+    </visual>
+    <collision name="rgbd_camera_collision">
+      <origin xyz="0 0 0" rpy="0 0 0"/>
+      <geometry>
+        <sphere radius="0.025" />
+      </geometry>
+    </collision>
+    <inertial>
+      <mass value="1e-5"/>
+      <origin xyz="0.0 0 0" rpy=" 0 0 0"/>
+      <inertia ixx="1e-6" ixy="0" ixz="0" iyy="1e-6" iyz="0" izz="1e-6" />
+    </inertial>
+  </link>
   <!-- LIDAR -->
   <joint name="hokuyo_joint" type="fixed">

Commit message: Fix Map My World project
Fixed RGBD camera so that mapping works correctly. Also added teleop.launch as per rubric.

File: my_robot/urdf/board_bot.xacro (robot description, xacro)
@@ -178,28 +178,10 @@
   </link>
  <!-- RGBD Camera -->
-  <joint name="rgbd_camera_optical_joint" type="fixed">
-    <origin xyz="0.5 0 -0.025" rpy="0 0 0"/>
-    <parent link="body"/>
-    <child link="rgbd_camera"/>
-    <axis xyz="0 1 0" rpy="0 0 0"/>
-  </joint>
-  <link name="rgbd_camera">
-    <visual name="rgbd_camera_visual">
-      <origin xyz="0 0 0" rpy="0 0 0"/>
-      <geometry>
-        <sphere radius="0.025" />
-      </geometry>
-    </visual>
-    <collision name="rgbd_camera_collision">
-      <origin xyz="0 0 0" rpy="0 0 0"/>
-      <geometry>
-        <sphere radius="0.025" />
-      </geometry>
-    </collision>
-    <inertial>
-      <mass value="1e-5"/>
-      <origin xyz="0.0 0 0" rpy=" 0 0 0"/>
-      <inertia ixx="1e-6" ixy="0" ixz="0" iyy="1e-6" iyz="0" izz="1e-6" />
-    </inertial>
+   <joint name="camera_optical_joint" type="fixed">
+    <origin xyz="0 0 0" rpy="-1.5707 0 -1.5707"/>
+    <parent link="camera"/>
+    <child link="camera_link_optical"/>
+  </joint>
+  <link name="camera_link_optical">
   </link>
   <!-- LIDAR -->
